File: hardware/base-usb-c.kicad_pcb (KiCad board)
At the start: 4 copper layers, 100 x 85 mm, 158 parts, among them J101 USB-A, J102 USB-C, J103 TNG-Power-TOP, J105 TNG-Data-TOP, P101 Debug, P102 PE, P202 PWR IN, SW101 BOOT, T201 744272251, U101 USB2517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

Commit message: version 1.1
 * fix usb-c cc resistors
Parts:
- R122, R123: value 56k -> 5k1
- turned R122 to 90 degrees
- turned R123 to 270 degrees
Connections:
- R122 pad 1: Net-(J102-Pad5) -> GND
- R122 pad 2: Net-(C141-Pad1) -> Net-(J102-Pad5)
- R123 pad 1: Net-(J102-Pad4) -> GND
- R123 pad 2: Net-(C141-Pad1) -> Net-(J102-Pad4)
Routing:
- net Net-(C141-Pad1): track 33.1 -> 31.0 mm
- net GND: track 838.3 -> 839.5 mm, vias 418 -> 420
Other:
- board text added: "Base USB-C REV 1.1"
- board text removed: "Base USB-C REV 1.0"

Commit message: add version 1.1
fix usb c
fix footprints
Parts:
- C139: footprint C0805 -> kicad-libraries:C0805E
- C205: footprint C1206 -> kicad-libraries:C0603F
- C208: footprint C0603F -> kicad-libraries:C0402F
- moved C205 0.77 mm to (92.4, 122.7)
- moved C208 0.23 mm to (93.1, 118.4)
Routing:
- net BOOT: track 68.4 -> 72.5 mm
- net GND: track 839.5 -> 841.7 mm, vias 420 -> 419
Other:
- board text added: "Copyright Tinkerforge GmbH 2020. This documentation describes Open Hardware and is licensed under the CERN OHL v. 1.1. You may redistribute and modify this documentation under the terms of the CERN OHL v.1.1. (http://ohwr.org/cernohl). This documentation is distributed WITHOUT ANY EXPRESS OR IMPLIED WARRANTY, INCLUDING OF MERCHANTABILITY, SATISFACTORY QUALITY AND FITNESS FOR A PARTICULAR PURPOSE.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"

Commit message: fix values
Parts:
- C108, C109, C117: value >100uF -> 100uF
- C121, C122: value TBD/47pF -> 47pF
- C137, C138: value TBD -> 33pF
- C203: value TBD -> 100µF
- C216, C219, C220: value >100µF -> 100µF
- X102: value TBD -> 8MHz

Commit message: fix value
Parts:
- C141: value >100uF -> 100uF
