File: hardware/base-usb-c.kicad_pcb (KiCad board)
At the start: 4 copper layers, 100 x 85 mm, 158 parts, among them J101 USB-A, J102 USB-C, J103 TNG-Power-TOP, J105 TNG-Data-TOP, P101 Debug, P102 PE, P202 PWR IN, SW101 BOOT, T201 744272251, U101 USB2517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

Commit message: fix footprint
Parts:
- R118: footprint kicad-libraries:1206 -> kicad-libraries:R1206
